File: PCBs/v1/References/ErgoWarrior_Final/ErgoWarrior_Final.kicad_pcb (KiCad board)
At the start: 2 copper layers, 76 x 57.5 mm, 26 parts

Commit message: Added finalised designs for v1.0.0
Parts:
- S1: value ~ -> Start
- S2: value ~ -> Select
- U1: value ~ -> Pi Pico
Other:
- board text added: "ErgoWarrior_v1.0.0"
- board text added: "I2C_Screen"
- board text added: "©2025 by kinpro1024"
