File: PCBs/v1/References/ErgoWarrior_Keys_Final/ErgoWarrior_Keys_Final.kicad_pcb (KiCad board)
At the start: 2 copper layers, 101 x 43.8 mm, 9 parts

Commit message: Added finalised designs for v1.0.0
Other:
- board text added: "ErgoWarrior_v1.0.0"
- board text added: "©2025 by kinpro1024"
Changed lines of the file:
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@@
 		(layer "Edge.Cuts")
+	)
+	(gr_text "©2025 by kinpro1024"
+		(at 121.92 92.71 0)
+		(layer "F.SilkS")
+		(effects
+			(font
+				(size 1.5 1.5)
+				(thickness 0.3)
+				(bold yes)
+			)
+			(justify left bottom)
+		)
+	)
+	(gr_text "ErgoWarrior_v1.0.0"
+		(at 108.966 77.978 0)
+		(layer "F.SilkS")
+		(effects
+			(font
+				(size 1.5 1.5)
+				(thickness 0.3)
+				(bold yes)
+			)
+			(justify left bottom)
+		)
 	)
 	(gr_text "B4"
@@
 			)
 			(justify mirror)
+		)
+	)
+	(gr_text "ErgoWarrior_v1.0.0"
+		(at 130.302 77.978 -0)
+		(layer "B.SilkS")
+		(effects
+			(font
+				(size 1.5 1.5)
+				(thickness 0.3)
+				(bold yes)
+			)
+			(justify left bottom mirror)
 		)
 	)
@@
 		)
 	)
+	(gr_text "©2025 by kinpro1024"
+		(at 148.082 92.71 -0)
+		(layer "B.SilkS")
+		(effects
+			(font
+				(size 1.5 1.5)
+				(thickness 0.3)
+				(bold yes)
+			)
+			(justify left bottom mirror)
+		)
+	)
